File: pcb/pcb.kicad_pcb (KiCad board)
At the start: 2 copper layers, 136 x 91.7 mm, 56 parts, among them J1 BATT, J2 BATT, SW1 SW_SPST, SW10 SW_SPST, SW11 SW_SPST, SW12 SW_SPST, SW13 SW_SPST, SW14 SW_SPST, SW15 SW_SPST, SW16 SW_SPST, SW17 SW_SPST, SW18 SW_SPST, SW19 SW_SPST, SW2 SW_SPST, SW20 SW_SPST, SW21 SW_SPST, SW3 SW_SPST, SW4 SW_SPST, SW5 SW_SPST, SW6 SW_SPST, SW7 SW_SPST, SW8 SW_SPST, SW9 SW_SPST, U1 XIAO_nRF52840

Commit message: Move the power switch to the side, change the hole for the switch to 5mm, move the little finger group down, cut a hole to access the controller power pins, enlarge the mounting hole to 5.5mm
Parts:
- removed H6, H7, H8: StandoffHole, one:Hole_2.2mm
- H1, H2, H3, H4: footprint one:Hole_4.2mm -> one:Hole_5.7mm
- moved PWR1 20.0 mm to (180.5, 55.9)
- moved D1 10.9 mm to (84.5, 86.9)
- moved D13 10.9 mm to (84.5, 107.9)
- moved D14 10.9 mm to (103.5, 107.9)
- moved D2 10.9 mm to (103.5, 86.9)
- moved D7 10.9 mm to (84.5, 88.9)
- moved D8 10.9 mm to (103.5, 88.9)
- moved H1 10.9 mm to (94.0, 87.4)
- moved H2 10.9 mm to (94.0, 106.4)
- moved SW1 10.9 mm to (84.5, 77.9)
- moved SW13 10.9 mm to (84.5, 115.9)
- moved SW14 10.9 mm to (103.5, 115.9)
- moved SW2 10.9 mm to (103.5, 77.9)
- moved SW7 10.9 mm to (84.5, 96.9)
- moved SW8 10.9 mm to (103.5, 96.9)
Routing:
- net Net-(J1-Pin_1): track 48.5 -> 91.8 mm, vias 5 -> 9
- net B+: track 17.7 -> 39.8 mm, vias 2 -> 3
- net C0: track 186.0 -> 202.0 mm
- net C1: track 164.4 -> 179.5 mm
- net R1: track 161.3 -> 174.7 mm
- net R2: track 175.6 -> 188.7 mm
- net B-: track 48.2 -> 60.4 mm
- net R0: track 165.5 -> 177.5 mm, vias 18 -> 17
- net C2: track 145.9 -> 152.7 mm
- net Net-(D2-A): track 14.0 -> 19.2 mm
- net Net-(D6-A): track 14.2 -> 19.3 mm
- net C3: track 160.6 -> 164.4 mm
- net C4: track 144.3 -> 147.4 mm
- net Net-(D14-A): track 24.6 -> 22.9 mm
- net Net-(D12-A): track 25.2 -> 23.9 mm
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Other:
- outline, holes or cut-outs redrawn
- board text added: "Ergonaut One v1.3 by yumagulovrn"
- board text removed: "Ergonaut One v1.2 by yumagulovrn"
